File: PCB/Navigator-BMS.kicad_pcb (KiCad board)
At the start: 2 copper layers, 48 parts, among them IC1 AP2112K, J1 Conn_01x03, J2 CAN, J3 CAN, Q1 IRF7480M, U1 BQ76920PW, U2 MCP2551-I-SN, U3 TMP117xxDRV, U4 STM32G441KBUx, U5 SN74AUP1T34DCK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

Commit message: Almost done with the layout, still want info on the mosfets the labs use + the battery connectors
Parts:
- moved J1 70.5 mm to (150.0, 83.2)
- moved U4 65.7 mm to (79.6, 52.9), turned to -90 degrees
- moved L1 53.9 mm to (80.5, 45.5)
- moved Q1 47.3 mm to (58.4, 42.9)
- moved U5 43.0 mm to (74.5, 55.2)
- moved C16 42.6 mm to (85.0, 44.7), turned to 90 degrees
- moved C17 36.4 mm to (87.5, 44.8), turned to -90 degrees
- moved R1 36.2 mm to (61.0, 48.8)
- moved U3 31.6 mm to (78.6, 58.6)
- moved C9 31.5 mm to (65.8, 44.8), turned to -90 degrees
- moved IC1 29.7 mm to (86.5, 50.5), turned to -90 degrees
- moved C4 29.2 mm to (62.5, 48.7), turned to -90 degrees
- moved C5 29.2 mm to (62.5, 50.7), turned to -90 degrees
- moved R6 27.8 mm to (61.0, 54.8)
- moved C8 27.7 mm to (62.0, 56.2), turned to 180 degrees
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Routing:
- net SRN: track 0.00 -> 11.7 mm
- net SRP: track 0.00 -> 9.63 mm
- net +14V: track 0.00 -> 5.01 mm
- net +BAT: track 0.00 -> 5.00 mm

Commit message: Layout Considerations + Schematic almost done
Parts:
- removed TP1, TP2, TP3, TP4: T, TestPoint:TestPoint_Pad_1.0x1.0mm
- added C18: 1uF, Capacitor_SMD:C_0402_1005Metric, F.Cu at (87.3, 43.4)
- added C19: 1uF, Capacitor_SMD:C_0402_1005Metric, F.Cu at (92.8, 43.3)
- added C20: 100nF, Capacitor_SMD:C_0402_1005Metric, F.Cu at (85.1, 51.8)
- added C21: 100nF, Capacitor_SMD:C_0402_1005Metric, F.Cu at (82.5, 54.3)
- added C22: 100nF, Capacitor_SMD:C_0402_1005Metric, F.Cu at (77.7, 49.4)
- added CELL 1: T, TestPoint:TestPoint_Pad_1.0x1.0mm, F.Cu at (51.2, 60.0)
- added CELL 2: T, TestPoint:TestPoint_Pad_1.0x1.0mm, F.Cu at (51.2, 58.0)
- added CELL 3: T, TestPoint:TestPoint_Pad_1.0x1.0mm, F.Cu at (51.2, 55.9)
- added CELL 4: T, TestPoint:TestPoint_Pad_1.0x1.0mm, F.Cu at (51.2, 53.9)
- added J4: Conn_01x05, Connector_JST:JST_EH_B5B-EH-A_1x05_P2.50mm_Vertical, F.Cu at (38.8, 39.7)
- C16, C17: footprint Capacitor_SMD:C_1206_3216Metric -> Capacitor_SMD:C_0805_2012Metric
- Q1: value IRF7480M -> SiSS27DN; footprint Package_DirectFET:DirectFET_ME -> Package_SO:Vishay_PowerPAK_1212-8_Single
- moved J1 62.4 mm to (103.3, 41.8), turned to 90 degrees
- moved C15 29.1 mm to (86.2, 35.2), turned to 180 degrees
- moved J2 20.0 mm to (102.2, 50.2), turned to 0 degrees
- moved C10 15.9 mm to (96.1, 50.5)
- moved J3 15.8 mm to (56.8, 32.8), turned to 0 degrees
- moved Q1 15.4 mm to (72.5, 36.7)
- moved R11 14.7 mm to (97.6, 51.0), turned to -90 degrees
- moved U5 14.0 mm to (86.0, 47.2)
- moved C12 9.14 mm to (74.8, 52.5), turned to -90 degrees
- moved U3 8.58 mm to (72.9, 52.2)
- moved C2 8.31 mm to (67.1, 56.9)
- moved R9 8.31 mm to (67.1, 54.9)
- moved C4 8.31 mm to (56.6, 54.6)
- moved C5 8.31 mm to (56.6, 56.6)
- moved C6 8.31 mm to (56.6, 58.6)
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Connections:
- Q1 pad 1: unconnected-(Q1-D-Pad1) -> GND
- Q1 pad 2: DSG -> GND
Routing:
- net SRN: track 11.7 -> 0.83 mm
- net PACK-: track 0.00 -> 9.77 mm
- net SRP: track 9.63 -> 0.74 mm
- net CELL3-F: track 0.00 -> 6.05 mm
- net CELL1-F: track 0.00 -> 5.67 mm
- net CELL2-F: track 0.00 -> 5.47 mm
- net CELL4-F: track 0.00 -> 4.85 mm
- net GND: track 0.00 -> 2.24 mm
- net Net-(U1-BAT): track 0.00 -> 1.78 mm
- net Net-(U1-CAP1): track 0.00 -> 1.74 mm
- net PACK+: track 0.00 -> 1.65 mm
