File: PCB/Navigator-BMS.kicad_sch (KiCad schematic)
At the start: 49 parts, among them IC1 AP2112K, J1 Conn_01x03, J2 CAN, J3 CAN, J4 Conn_01x05, Q1 IRF7480M, U1 BQ76920PW, U2 MCP2551-I-SN, U3 TMP117xxDRV, U4 STM32G441KBUx, U5 SN74AUP1T34DCK, U6 TPS

Commit message: Layout Considerations + Schematic almost done
Parts:
- removed Q1: IRF7480M, Package_DirectFET:DirectFET_ME, symbol Transistor_FET:IRF7480M
- added C18, C19: 1uF, Capacitor_SMD:C_0402_1005Metric, symbol Device:C
- added C20, C21, C22: 100nF, Capacitor_SMD:C_0402_1005Metric, symbol Device:C
- added Q1: SiSS27DN, Package_SO:Vishay_PowerPAK_1212-8_Single, symbol Transistor_FET:SiSS27DN
- added TP5: T, TestPoint:TestPoint_Pad_1.0x1.0mm, symbol Connector:TestPoint
- C16, C17: footprint Capacitor_SMD:C_1206_3216Metric -> Capacitor_SMD:C_0805_2012Metric
- J4: footprint (none) -> Connector_JST:JST_EH_B5B-EH-A_1x05_P2.50mm_Vertical
Connections:
- net +3.3V: now also C19.1, C20.1, C21.1, C22.1
- net +5V: now also C18.1
- net CELL1: now also TP4.1
- net CELL2: now also TP3.1
- net CELL3: now also TP2.1
- net CELL4: now also TP1.1
- net DSG: now also Q1.4 (G)
- net GND: now also C18.2, C19.2, C20.2, C21.2, C22.2, Q1.1 (S), Q1.2 (S), Q1.3 (S), TP5.1
- new net Load: Q1.5 (D)
Other:
- moved on the sheet: IC1, J1, J2, J3, J4, TP1, TP2, TP3, TP4, U5

Commit message: Finished layout. Board Shape kinda chopped but will be edited. Analog section far away from high current areas!
Parts:
- removed C1, C9: 100nF, Capacitor_SMD:C_0402_1005Metric, symbol Device:C
- removed IC1: AP2112K, Custom-Footprints:SOT95P285X140-5N, symbol Custom-Symbols:AP2112
- removed U4: STM32G441KBUx, Package_DFN_QFN:QFN-32-1EP_5x5mm_P0.5mm_EP3.45x3.45mm, symbol MCU_ST_STM32G4:STM32G441KBUx
- added C11, C18, C20, C24: 100nF, Capacitor_SMD:C_0402_1005Metric, symbol Device:C
- added IC1: INA236AIDDFR, Custom-Footprints:SOP65P280X110-8N, symbol Custom-Symbols:INA236AIDDFR
- added R16, R17: 4.7k, Resistor_SMD:R_0402_1005Metric, symbol Device:R
- added U3: AMS1117-3.3, Package_TO_SOT_SMD:SOT-223-3_TabPin2, symbol Regulator_Linear:AMS1117-3.3
- added U5: STM32G441CBTx, Package_QFP:LQFP-48_7x7mm_P0.5mm, symbol MCU_ST_STM32G4:STM32G441CBTx
- C15: renamed from C18; value 1uF -> 10uF; footprint Capacitor_SMD:C_0402_1005Metric -> Capacitor_SMD:C_0805_2012Metric
- C19: value 1uF -> 10uF; footprint Capacitor_SMD:C_0402_1005Metric -> Capacitor_SMD:C_0805_2012Metric
- R10: value 4.7k -> 0
- renumbered C2 to C1, C12 to C10, C20 to C12, C21 to C13, C13 to C14, C22 to C16, C14 to C17, C3 to C2, C15 to C21, C16 to C22, C17 to C23, C4 to C3, C5 to C4, C6 to C5, C7 to C6, C8 to C7, C10 to C8, C11 to C9, TP4 to CEEL1, TP3 to CELL2, TP2 to CELL3, TP1 to CELL4, TP5 to GND1, U3 to IC2, U6 to IC3, J3 to J1, J4 to J2, J2 to J3, J1 to J4, R8 to R5, R5 to R8, U5 to U4
Connections:
- net +3.3V: now also C11.1, C18.1, C20.1, C24.1, IC1.4 (VS), R16.1, R17.1, U3.2 (VO), U5.1 (VBAT), U5.21 (VDDA), U5.24 (VDD), U5.36 (VDD), U5.48 (VDD)
- net +5V: now also U3.3 (VI)
- net GND: now also C11.2, C18.2, C20.2, C24.2, IC1.3 (GND), IC1.7 (A0), U3.1 (GND), U5.19 (VSSA), U5.23 (VSS), U5.35 (VSS), U5.47 (VSS)
- net I2C-SCL-1: now also IC1.5 (SCL), R17.2, U5.31 (PA9)
- net I2C-SDA-1: now also IC1.6 (SDA), R16.2, U5.30 (PA8)
- net SWD-SWCLK: now also U5.38 (PA14)
- net SWD-SWDIO: now also U5.39 (PA15)
- net TMP117-ALERT: now also U5.17 (PB1)
- net SRN: no longer names the net of U1.19 (SRN)
- net SRN: no longer R8.1
- net SRP: no longer names the net of U1.18 (SRP)
- net SRP: no longer R5.1
- new net INA236-ALERT: IC1.8 (~{ALERT}), U5.16 (PB0)
- new net SHUNT+: IC1.1 (IN+), R5.1
- new net SHUNT-: IC1.2 (IN-), R8.1
- no-connect marks 4 -> 6
Other:
- moved on the sheet: C12, C13, C15, C16, C19, C8, C9, CEEL1, CELL2, CELL3, CELL4, GND1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

Commit message: Layout complete. Waiting to order + starting firmware using Russel's BQ76920 Test Board
Parts:
- removed C14, C17: 22uF, Capacitor_SMD:C_0805_2012Metric, symbol Device:C
- removed C21: 33pF, Capacitor_SMD:C_0402_1005Metric, symbol Device:C
- removed C22: 47uF, Capacitor_SMD:C_0805_2012Metric, symbol Device:C
- removed IC3: TPS, Custom-Footprints:SOTFL50P160X60-6N, symbol Custom-Symbols:TPS565242DRLR
- removed Q1: SiSS27DN, Package_SO:Vishay_PowerPAK_1212-8_Single, symbol Transistor_FET:SiSS27DN
- removed R13: 1k, Resistor_SMD:R_0402_1005Metric, symbol Device:R
- added C1, C2: 22uF, Capacitor_SMD:C_0805_2012Metric, symbol Device:C
- added C24: 30pF, Capacitor_SMD:C_0402_1005Metric, symbol Device:C
- added C28: 4.7uF, Capacitor_SMD:C_0603_1608Metric, symbol Device:C
- added C3: 100nF, Capacitor_SMD:C_0402_1005Metric, symbol Device:C
- added C4, C5: 47uF, Capacitor_SMD:C_0805_2012Metric, symbol Device:C
- added C7: 10nF, Capacitor_SMD:C_0402_1005Metric, symbol Device:C
- added H1: M1, MountingHole:MountingHole_3.2mm_M3_Pad_Via, symbol Mechanical:MountingHole_Pad
- added H2: M2, MountingHole:MountingHole_3.2mm_M3_Pad_Via, symbol Mechanical:MountingHole_Pad
- added H3: M3, MountingHole:MountingHole_3.2mm_M3_Pad_Via, symbol Mechanical:MountingHole_Pad
- added H4: M4, MountingHole:MountingHole_3.2mm_M3_Pad_Via, symbol Mechanical:MountingHole_Pad
- added J4: CAN, Connector_AMASS:AMASS_XT60-F_1x02_P7.20mm_Vertical, symbol Connector_Generic:Conn_01x02
- added J6: Conn_01x04, Connector_PinSocket_2.54mm:PinSocket_1x04_P2.54mm_Vertical, symbol Connector_Generic:Conn_01x04
- added Q1: NTMFS016N06CT1G, Package_SO:ONSemi_SO-8FL_488AA, symbol Transistor_FET:NTMFS016N06CT1G
- added R1: 47k, Resistor_SMD:R_0402_1005Metric, symbol Device:R
- added R2: 220k, Resistor_SMD:R_0402_1005Metric, symbol Device:R
- added R21: 4.7k, Resistor_SMD:R_0402_1005Metric, symbol Device:R
- added R3: 10k, Resistor_SMD:R_0402_1005Metric, symbol Device:R
- added R4: 30k, Resistor_SMD:R_0402_1005Metric, symbol Device:R
- added U1: TPS566238RQFR, Custom-Footprints:TPS566238RQFR, symbol Custom-Symbols:TPS566238RQFR
- added Y1: Crystal_GND24, Crystal:Crystal_SMD_3225-4Pin_3.2x2.5mm, symbol Device:Crystal_GND24
- C23: value 47uF -> 30pF; footprint Capacitor_SMD:C_0805_2012Metric -> Capacitor_SMD:C_0402_1005Metric
- J1: renamed from J2; footprint Connector_JST:JST_EH_B5B-EH-A_1x05_P2.50mm_Vertical -> Connector_PinHeader_2.54mm:PinHeader_1x05_P2.54mm_Vertical
- L1: value 2.2uH -> L; footprint Inductor_SMD:L_Coilcraft_XAL5030-XXX -> Inductor_SMD:L_Coilcraft_XAL4020-XXX
- R12: value 4.7k -> 1M; footprint Resistor_SMD:R_0402_1005Metric -> Resistor_SMD:R_0603_1608Metric
- R14: value 220k -> 4.7k
- R15: value 30k -> 4.7k
- renumbered C19 to C10, C3 to C12, C4 to C13, C5 to C14, C6 to C15, C7 to C16, C12 to C17, C13 to C18, C16 to C19, C18 to C20, C20 to C21, C8 to C22, C2 to C25, C9 to C26, C24 to C27, C10 to C6, C1 to C8, C15 to C9, CELL4 to CELL1, CELL3 to CELL2, CELL2 to CELL3, IC2 to IC1, IC1 to IC2, J4 to J2, J1 to J3, J3 to J5, R3 to R10, R4 to R11, R6 to R13, R7 to R16, R11 to R17, R10 to R18, R5 to R19, R8 to R20, R9 to R5, R1 to R6, R16 to R7, R17 to R8, R2 to R9, U1 to U2, U5 to U4, U4 to U5, U2 to U6
Connections:
- net BAT+ is gone; now on net +BAT: J3.2 (Pin_2)
- net PACK+ is gone; now on net +14V: R5.2, U2.9 (REGSRC)
- net +14V: now also C1.1, C2.1, J4.2 (Pin_2), R1.1, U1.5 (VIN), U1.6 (VIN); no longer R12.1
- net +3.3V: now also R14.1, R15.1, U4.20 (VREF+), C28.1, J6.4 (Pin_4)
- net +5V: now also J2.3 (Pin_3), C4.1, C5.1, R2.1; no longer C23.1, J2.1 (Pin_1), R14.1
- net BQ76920-ALERT: now also U4.40 (PB3)
- net CAN-RX: now also U4.33 (PA11)
- net CAN-TX: now also U4.34 (PA12)
- net DSG: now also R12.1, Q1.4 (G)
- net GND: now also J2.1 (Pin_1), R12.2, C1.2, C2.2, C24.2, C28.2, C4.2, C5.2, C7.1, H1.1, H2.1, H3.1, H4.1, J6.3 (Pin_3), Q1.1 (S), Q1.2 (S), Q1.3 (S), R21.1, R3.2, R4.2, U1.4 (PGND), Y1.2 (G), Y1.4 (G); no longer C15.2, C16.1, GND1.1, J1.5 (Pin_5), J2.3 (Pin_3), R13.1, R15.2
- net I2C-SCL-1: now also U4.39 (PA15); no longer U4.31 (PA9)
- net I2C-SDA-1: now also U4.44 (PB7); no longer U4.30 (PA8)
- net INA236-ALERT: now also R14.2, U4.2 (PC13); no longer U4.16 (PB0)
- net LED-3.3V: now also U4.14 (PA6)
- net Load: now also J4.1 (Pin_1), Q1.5 (D)
- net SWD-SWCLK: now also J6.1 (Pin_1)
- net SWD-SWDIO: now also U4.37 (PA13), J6.2 (Pin_2); no longer U4.39 (PA15)
- net TMP117-ALERT: now also R15.2, U4.13 (PA5); no longer U4.17 (PB1)
- net at L1.1: now also C3.2, U1.8 (SW)
- net BQ76920-BOOT: now reaches U2.6 (TS1)
- net BQ76920-BOOT: now also U4.41 (PB4)
- net at U4.45 (PB8): now also R21.2
- net RCC-IN: now reaches U4.5 (PF0)
- net RCC-IN: now also C24.1, Y1.3
- net RCC-OUT: now reaches U4.6 (PF1)
- net RCC-OUT: now also C23.1, Y1.1
- net CAN-H renamed CAN+
- net CAN-L renamed CAN-
- new net: C7.2, U1.9 (SS)
- new net: C3.1, U1.7 (BST)
- new net: R2.2, R4.1, U1.2 (FB)
- new net: R1.2, R3.1, U1.3 (EN)
- new net CELL0: C15.2, C16.1, GND1.1, J1.5 (Pin_5), R13.1
- no-connect marks 6 -> 30
Other:
- moved on the sheet: C11, IC2
